File: cad/uDuino.brd (EAGLE design)
At the start: 86.4 x 26 mm, 23 parts, among them IC1 LM7805, IC2 ATMEGA328, J1 POWER_JACK", Q1 16MHZ

Commit message: Adding project to kitnic.it
Parts:
- renumbered U$1 to JP5
Changed lines of the file:
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@@
 <element name="J1" library="RBBB" package="POWER_JACK" value="POWER_JACK&quot;" x="80.645" y="24.765" smashed="yes" rot="R180"/>
 <element name="D1" library="adafruit" package="DO41-10" value="1N4004" x="62.865" y="11.43" smashed="yes" rot="R90"/>
-<element name="U$1" library="RBBB" package="1X02_HEADER" value="1X02_HEADER" x="73.025" y="22.225" rot="R90"/>
+<element name="JP5" library="RBBB" package="1X02_HEADER" value="1X02_HEADER" x="73.025" y="22.225" rot="R90"/>
 <element name="IC2" library="RBBB" package="ATMEGA328" value="ATMEGA328" x="32.385" y="15.875" smashed="yes"/>
 <element name="C3" library="RBBB" package="UNPOLARIZED_CAP" value="0.1uF" x="67.31" y="23.495" smashed="yes"/>
@@
 <contactref element="J1" pad="PWR"/>
 <contactref element="D1" pad="C"/>
-<contactref element="U$1" pad="1"/>
+<contactref element="JP5" pad="1"/>
 <wire x1="80.645" y1="11.065" x2="74.025" y2="4.445" width="0.4064" layer="1"/>
 <wire x1="72.39" y1="4.445" x2="74.025" y2="4.445" width="0.4064" layer="1"/>
@@
 <contactref element="J1" pad="GND"/>
 <contactref element="D1" pad="A"/>
-<contactref element="U$1" pad="2"/>
+<contactref element="JP5" pad="2"/>
 <contactref element="IC2" pad="22"/>
 <contactref element="IC2" pad="8"/>
