File: cad/uDuino.sch (EAGLE design)
At the start: 23 parts, among them IC1 LM7805, IC2 ATMEGA328, J1 POWER_JACK", Q1 16MHZ

Commit message: Adding project to kitnic.it
Parts:
- renumbered U$1 to JP5
Changed lines of the file:
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@@
 <part name="J1" library="RBBB" deviceset="POWER_JACK" device="&quot;"/>
 <part name="D1" library="adafruit" deviceset="1N4004" device=""/>
-<part name="U$1" library="RBBB" deviceset="1X02_HEADER" device=""/>
+<part name="JP5" library="RBBB" deviceset="1X02_HEADER" device=""/>
 <part name="IC2" library="RBBB" deviceset="ATMEGA328" device="&quot;" value="ATMEGA328"/>
 <part name="GND2" library="RBBB" deviceset="SUPPLY_GND" device=""/>
@@
 <instance part="J1" gate="G$1" x="-17.78" y="-10.16"/>
 <instance part="D1" gate="1" x="0" y="-15.24" rot="R90"/>
-<instance part="U$1" gate="G$1" x="-5.08" y="12.7" rot="R90"/>
+<instance part="JP5" gate="G$1" x="-5.08" y="12.7" rot="R90"/>
 <instance part="IC2" gate="G$1" x="22.86" y="91.44"/>
 <instance part="GND2" gate="1" x="-27.94" y="48.26"/>
@@
 <wire x1="0" y1="-12.7" x2="0" y2="-2.54" width="0.1524" layer="91"/>
 <junction x="0" y="-2.54"/>
-<pinref part="U$1" gate="G$1" pin="1"/>
+<pinref part="JP5" gate="G$1" pin="1"/>
 <wire x1="-7.62" y1="5.08" x2="-7.62" y2="-2.54" width="0.1524" layer="91"/>
 <junction x="-7.62" y="-2.54"/>
@@
 <wire x1="0" y1="-17.78" x2="0" y2="-25.4" width="0.1524" layer="91"/>
 <junction x="0" y="-25.4"/>
-<pinref part="U$1" gate="G$1" pin="2"/>
+<pinref part="JP5" gate="G$1" pin="2"/>
 <wire x1="-5.08" y1="5.08" x2="-5.08" y2="-25.4" width="0.1524" layer="91"/>
 <junction x="-5.08" y="-25.4"/>
